File: hardware/signal-to-can/can_transciever_no_term.kicad_sch (KiCad schematic)
At the start: 6 parts

Commit message: 1st rev PCB layout
Parts:
- gave numbers to parts that had none: 6
Changed lines of the file:
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@@
 		(dnp no)
 		(fields_autoplaced yes)
-		(property "Reference" "TP?"
+		(property "Reference" "TP5"
 			(at 144.78 112.5219 0)
 			(effects
@@
 			(project "can_transciever_no_term"
 				(path "/742f64ac-c4d8-4561-a2a9-e0e3f6f67ce8/b93d8d5a-c9dc-4552-9959-3cf22fd198ac"
-					(reference "TP?")
+					(reference "TP5")
 					(unit 1)
 				)
@@
 		(dnp no)
 		(fields_autoplaced yes)
-		(property "Reference" "#PWR?"
+		(property "Reference" "#PWR030"
 			(at 162.56 88.9 0)
 			(effects
@@
 			(project "can_transciever_no_term"
 				(path "/742f64ac-c4d8-4561-a2a9-e0e3f6f67ce8/b93d8d5a-c9dc-4552-9959-3cf22fd198ac"
-					(reference "#PWR?")
+					(reference "#PWR030")
 					(unit 1)
 				)
@@
 		(dnp no)
 		(fields_autoplaced yes)
-		(property "Reference" "#PWR?"
+		(property "Reference" "#PWR028"
 			(at 157.48 77.47 0)
 			(effects
@@
 			(project "can_transciever_no_term"
 				(path "/742f64ac-c4d8-4561-a2a9-e0e3f6f67ce8/b93d8d5a-c9dc-4552-9959-3cf22fd198ac"
-					(reference "#PWR?")
+					(reference "#PWR028")
 					(unit 1)
 				)
@@
 	)
 	(symbol
+		(lib_name "GND_3")
 		(lib_id "power:GND")
 		(at 193.04 101.6 90)
@@
 		(dnp no)
 		(fields_autoplaced yes)
-		(property "Reference" "#PWR?"
+		(property "Reference" "#PWR031"
 			(at 199.39 101.6 0)
 			(effects
@@
 			(project "can_transciever_no_term"
 				(path "/742f64ac-c4d8-4561-a2a9-e0e3f6f67ce8/b93d8d5a-c9dc-4552-9959-3cf22fd198ac"
-					(reference "#PWR?")
+					(reference "#PWR031")
 					(unit 1)
 				)
@@
 		(on_board yes)
 		(dnp no)
-		(property "Reference" "U?"
+		(property "Reference" "U3"
 			(at 149.86 91.44 0)
 			(effects
@@
 			(project "can_transciever_no_term"
 				(path "/742f64ac-c4d8-4561-a2a9-e0e3f6f67ce8/b93d8d5a-c9dc-4552-9959-3cf22fd198ac"
-					(reference "U?")
+					(reference "U3")
 					(unit 1)
 				)
@@
 	)
 	(symbol
+		(lib_name "+3.3V_1")
 		(lib_id "power:+3.3V")
 		(at 144.78 81.28 0)
@@
 		(dnp no)
 		(fields_autoplaced yes)
-		(property "Reference" "#PWR?"
+		(property "Reference" "#PWR027"
 			(at 144.78 85.09 0)
 			(effects
@@
 			(project "can_transciever_no_term"
 				(path "/742f64ac-c4d8-4561-a2a9-e0e3f6f67ce8/b93d8d5a-c9dc-4552-9959-3cf22fd198ac"
-					(reference "#PWR?")
+					(reference "#PWR027")
 					(unit 1)
 				)
@@
 		(dnp no)
 		(fields_autoplaced yes)
-		(property "Reference" "C?"
+		(property "Reference" "C14"
 			(at 138.43 85.0962 0)
 			(effects
@@
 			(project "can_transciever_no_term"
 				(path "/742f64ac-c4d8-4561-a2a9-e0e3f6f67ce8/b93d8d5a-c9dc-4552-9959-3cf22fd198ac"
-					(reference "C?")
+					(reference "C14")
 					(unit 1)
 				)
@@
 	)
 	(symbol
+		(lib_name "GND_2")
 		(lib_id "power:GND")
 		(at 157.48 115.57 0)
@@
 		(dnp no)
 		(fields_autoplaced yes)
-		(property "Reference" "#PWR?"
+		(property "Reference" "#PWR029"
 			(at 157.48 121.92 0)
 			(effects
@@
 			(project "can_transciever_no_term"
 				(path "/742f64ac-c4d8-4561-a2a9-e0e3f6f67ce8/b93d8d5a-c9dc-4552-9959-3cf22fd198ac"
-					(reference "#PWR?")
+					(reference "#PWR029")
 					(unit 1)
 				)
@@
 	)
 	(symbol
+		(lib_name "GND_1")
 		(lib_id "power:GND")
 		(at 135.89 90.17 0)
@@
 		(dnp no)
 		(fields_autoplaced yes)
-		(property "Reference" "#PWR?"
+		(property "Reference" "#PWR026"
 			(at 135.89 96.52 0)
 			(effects
@@
 			(project "can_transciever_no_term"
 				(path "/742f64ac-c4d8-4561-a2a9-e0e3f6f67ce8/b93d8d5a-c9dc-4552-9959-3cf22fd198ac"
-					(reference "#PWR?")
+					(reference "#PWR026")
 					(unit 1)
 				)
@@
 		(dnp no)
 		(fields_autoplaced yes)
-		(property "Reference" "C?"
+		(property "Reference" "C15"
 			(at 165.1 77.4762 0)
 			(effects
@@
 			(project "can_transciever_no_term"
 				(path "/742f64ac-c4d8-4561-a2a9-e0e3f6f67ce8/b93d8d5a-c9dc-4552-9959-3cf22fd198ac"
-					(reference "C?")
+					(reference "C15")
 					(unit 1)
 				)
@@
 		(on_board yes)
 		(dnp no)
-		(property "Reference" "D?"
+		(property "Reference" "D4"
 			(at 187.198 89.154 90)
 			(effects
@@
 			(project "can_transciever_no_term"
 				(path "/742f64ac-c4d8-4561-a2a9-e0e3f6f67ce8/b93d8d5a-c9dc-4552-9959-3cf22fd198ac"
-					(reference "D?")
+					(reference "D4")
 					(unit 1)
 				)
@@
 		(dnp no)
 		(fields_autoplaced yes)
-		(property "Reference" "TP?"
+		(property "Reference" "TP4"
 			(at 133.35 112.5219 0)
 			(effects
@@
 			(project "can_transciever_no_term"
 				(path "/742f64ac-c4d8-4561-a2a9-e0e3f6f67ce8/b93d8d5a-c9dc-4552-9959-3cf22fd198ac"
-					(reference "TP?")
-					(unit 1)
-				)
+					(reference "TP4")
+					(unit 1)
+				)
