File: hardware/signal-to-can/stm32f042k6ux.kicad_sch (KiCad schematic)
At the start: 20 parts, among them J3 TC2030, U5 STM32F042K6Ux, Y2 ECS-160-10-36Q-AES-TR

Commit message: 1st rev PCB layout
Parts:
- renumbered C17 to C1, C26 to C10, C18 to C2, C19 to C3, C20 to C4, C21 to C5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
Connections:
- net 3.3V_ANALOG_INPUT_8 is gone; now on net LED_STATUS_1: U1.14 (PB0)
- net 3.3V_ANALOG_INPUT_9 is gone; now on net LED_STATUS_2: U1.15 (PB1)
- net LED_STATUS_1: no longer U1.16 (PB2)
- net LED_STATUS_2: no longer U1.26 (PB3)
- no-connect marks 1 -> 11
