File: hardware/signal-to-can/stm32f042k6ux.kicad_sch (KiCad schematic)
At the start: 20 parts, among them J2 TC2030, U1 STM32F042K6Ux, Y1 ECS-160-10-36Q-AES-TR

Commit message: Working CAN peripheral
- heartbeat
- test can message
- adc module compiling
Other:
- note added: "BOOT0 to 3V3: Boot to system memory BOOT0 to GND: Boot to flash memory"
Changed lines of the file:
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@@
 	(generator_version "9.0")
 	(paper "A4")
+	(text "BOOT0 to 3V3: Boot to system memory\nBOOT0 to GND: Boot to flash memory"
+		(exclude_from_sim no)
+		(at 35.56 141.986 0)
+		(effects
+			(font
+				(size 1.27 1.27)
+			)
+		)
+	)
 	(text "Microcontroller"
 		(exclude_from_sim no)
