File: hardware/signal-to-can/switching_regulator_5V_500ma_28V_input.kicad_sch (KiCad schematic)
At the start: 7 parts, among them U1 R-78E5.0-0.5

Commit message: 1st rev PCB layout
Parts:
- C16: renamed from C1; footprint (none) -> Capacitor_SMD:C_0603_1608Metric
- C17: renamed from C2; footprint (none) -> Capacitor_SMD:C_0603_1608Metric
- D21: renamed from D20; footprint Diode_THT:D_DO-41_SOD81_P10.16mm_Horizontal -> Diode_SMD:D_SOD-123
- TP6: renamed from TP2; footprint (none) -> TestPoint:TestPoint_Pad_D1.0mm
- renumbered D19 to D22, R1 to R14, U1 to U4
Changed lines of the file:
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@@
 		(dnp no)
 		(fields_autoplaced yes)
-		(property "Reference" "#PWR034"
+		(property "Reference" "#PWR067"
 			(at 176.53 87.63 0)
 			(effects
@@
 			(project ""
 				(path "/742f64ac-c4d8-4561-a2a9-e0e3f6f67ce8/1302be3c-854e-4381-9e1e-22325ed48fb8"
-					(reference "#PWR034")
+					(reference "#PWR067")
 					(unit 1)
 				)
@@
 		(on_board yes)
 		(dnp no)
-		(property "Reference" "C2"
+		(property "Reference" "C17"
 			(at 162.56 90.1762 0)
 			(effects
@@
 			)
 		)
-		(property "Footprint" ""
+		(property "Footprint" "Capacitor_SMD:C_0603_1608Metric"
 			(at 160.02 91.44 0)
 			(effects
@@
 			(project "signal-to-can"
 				(path "/742f64ac-c4d8-4561-a2a9-e0e3f6f67ce8/1302be3c-854e-4381-9e1e-22325ed48fb8"
-					(reference "C2")
+					(reference "C17")
 					(unit 1)
 				)
@@
 		(dnp no)
 		(fields_autoplaced yes)
-		(property "Reference" "TP2"
+		(property "Reference" "TP6"
 			(at 170.18 80.5179 0)
 			(effects
@@
 			)
 		)
-		(property "Footprint" ""
+		(property "Footprint" "TestPoint:TestPoint_Pad_D1.0mm"
 			(at 172.72 85.09 0)
 			(effects
@@
 			(project ""
 				(path "/742f64ac-c4d8-4561-a2a9-e0e3f6f67ce8/1302be3c-854e-4381-9e1e-22325ed48fb8"
-					(reference "TP2")
+					(reference "TP6")
 					(unit 1)
 				)
@@
 		(dnp no)
 		(fields_autoplaced yes)
-		(property "Reference" "#PWR035"
+		(property "Reference" "#PWR064"
 			(at 124.46 87.63 0)
 			(effects
@@
 			(project ""
 				(path "/742f64ac-c4d8-4561-a2a9-e0e3f6f67ce8/1302be3c-854e-4381-9e1e-22325ed48fb8"
-					(reference "#PWR035")
+					(reference "#PWR064")
 					(unit 1)
 				)
@@
 		(dnp no)
 		(fields_autoplaced yes)
-		(property "Reference" "U1"
+		(property "Reference" "U4"
 			(at 148.59 81.28 0)
 			(effects
@@
 			(project ""
 				(path "/742f64ac-c4d8-4561-a2a9-e0e3f6f67ce8/1302be3c-854e-4381-9e1e-22325ed48fb8"
-					(reference "U1")
+					(reference "U4")
 					(unit 1)
 				)
@@
 		(dnp no)
 		(fields_autoplaced yes)
-		(property "Reference" "#PWR033"
+		(property "Reference" "#PWR065"
 			(at 143.51 106.68 0)
 			(effects
@@
 			(project ""
 				(path "/742f64ac-c4d8-4561-a2a9-e0e3f6f67ce8/1302be3c-854e-4381-9e1e-22325ed48fb8"
-					(reference "#PWR033")
+					(reference "#PWR065")
 					(unit 1)
 				)
@@
 		(dnp no)
 		(fields_autoplaced yes)
-		(property "Reference" "D20"
+		(property "Reference" "D21"
 			(at 127.3175 81.28 0)
 			(effects
@@
 			)
 		)
-		(property "Footprint" "Diode_THT:D_DO-41_SOD81_P10.16mm_Horizontal"
+		(property "Footprint" "Diode_SMD:D_SOD-123"
 			(at 127 83.185 0)
 			(effects
@@
 			(project ""
 				(path "/742f64ac-c4d8-4561-a2a9-e0e3f6f67ce8/1302be3c-854e-4381-9e1e-22325ed48fb8"
-					(reference "D20")
+					(reference "D21")
 					(unit 1)
 				)
@@
 		(dnp no)
 		(fields_autoplaced yes)
-		(property "Reference" "D19"
+		(property "Reference" "D22"
 			(at 176.53 101.9174 90)
 			(effects
@@
 			(project "signal-to-can"
 				(path "/742f64ac-c4d8-4561-a2a9-e0e3f6f67ce8/1302be3c-854e-4381-9e1e-22325ed48fb8"
-					(reference "D19")
+					(reference "D22")
 					(unit 1)
 				)
@@
 		(dnp no)
 		(fields_autoplaced yes)
-		(property "Reference" "#PWR050"
+		(property "Reference" "#PWR066"
 			(at 172.72 113.03 0)
 			(effects
@@
 			(project "signal-to-can"
 				(path "/742f64ac-c4d8-4561-a2a9-e0e3f6f67ce8/1302be3c-854e-4381-9e1e-22325ed48fb8"
-					(reference "#PWR050")
+					(reference "#PWR066")
 					(unit 1)
 				)
@@
 		(dnp no)
 		(fields_autoplaced yes)
-		(property "Reference" "R1"
+		(property "Reference" "R14"
 			(at 175.26 91.4399 0)
 			(effects
@@
 			(project "signal-to-can"
 				(path "/742f64ac-c4d8-4561-a2a9-e0e3f6f67ce8/1302be3c-854e-4381-9e1e-22325ed48fb8"
-					(reference "R1")
+					(reference "R14")
 					(unit 1)
 				)
@@
 		(on_board yes)
 		(dnp no)
-		(property "Reference" "C1"
+		(property "Reference" "C16"
 			(at 134.62 90.1762 0)
 			(effects
@@
 			)
 		)
-		(property "Footprint" ""
+		(property "Footprint" "Capacitor_SMD:C_0603_1608Metric"
 			(at 137.16 91.44 0)
 			(effects
@@
 			(project ""
 				(path "/742f64ac-c4d8-4561-a2a9-e0e3f6f67ce8/1302be3c-854e-4381-9e1e-22325ed48fb8"
-					(reference "C1")
-					(unit 1)
-				)
+					(reference "C16")
+					(unit 1)
+				)
