File: hardware/signal-to-can/signal-to-can.kicad_pcb (KiCad board)
At the start: 2 copper layers, 70 x 55 mm, 79 parts, among them J1 AMP_Superseal_9-6437287-8, J2 TC2030, U1 STM32F042K6Ux, U2 TLE42744DV33ATMA1, U3 TCAN3403DRQ1, U4 R-78E5.0-0.5, Y1 ECS-160-10-36Q-AES-TR

Commit message: production v1
Connections:
- J1 pad 17: +3.3V -> +3V3
- J1 pad 18: +3.3V -> +3V3
- J1 pad 19: +3.3V -> +3V3
Routing:
- net +3V3: track 211.1 -> 263.7 mm, vias 21 -> 23
- net +BATT: track 36.8 -> 58.2 mm, vias 0 -> 2
- net +5V: track 40.0 -> 60.4 mm
- net GND: track 61.7 -> 82.1 mm
- net +3.3V: track 6.00 -> 0.00 mm
Other:
- board text added: "0"
- board text added: "1"
- board text added: "2"
- board text added: "3"
- board text added: "3V3"
- board text added: "4"
- board text added: "5"
- board text added: "5V"
- board text added: "6"
- board text added: "7"
- board text added: "8x analog inputs 0 - 12V 10mV resolution 5V 0.5mA sensor power 3.3V 250mA sensor power"
- board text added: "BATT"
- board text added: "BRG 7/25"
- board text added: "GND"
- board text added: "SIGNAL TO CAN"
